Commit message: add odrive_diffbot demo

File: odrive_demo_description/urdf/odrive.ros2_control.xacro (robot description, xacro)
@@ -1,5 +1,6 @@
 <?xml version="1.0"?>
 <robot xmlns:xacro="http://www.ros.org/wiki/xacro">
-  <xacro:macro name="odrive_ros2_control" params="name enable_joint0:=^|true enable_joint1:=^|true">
+  <xacro:macro name="odrive_ros2_control"
+    params="name serial_number:=^|000000000000 enable_joint0:=^|true enable_joint1:=^|true joint0_name:=^|joint0 joint1_name:=^|joint1">
     <ros2_control name="${name}" type="system">
       <hardware>
@@ -7,9 +8,9 @@
       </hardware>
       <sensor name="odrv0">
-        <param name="serial_number">000000000000</param>
+        <param name="serial_number">${serial_number}</param>
       </sensor>
       <xacro:if value="${enable_joint0}">
-        <joint name="joint0">
-          <param name="serial_number">000000000000</param>
+        <joint name="${joint0_name}">
+          <param name="serial_number">${serial_number}</param>
           <param name="axis">0</param>
           <param name="enable_watchdog">1</param>
@@ -18,6 +19,6 @@
       </xacro:if>
       <xacro:if value="${enable_joint1}">
-        <joint name="joint1">
-          <param name="serial_number">000000000000</param>
+        <joint name="${joint1_name}">
+          <param name="serial_number">${serial_number}</param>
           <param name="axis">1</param>
           <param name="enable_watchdog">1</param>

Commit message: motor direction change

File: odrive_demo_description/urdf/odrive.ros2_control.xacro (robot description, xacro)
@@ -15,5 +15,5 @@
           <param name="axis">0</param>
           <param name="enable_watchdog">1</param>
-          <param name="watchdog_timeout">0.1</param>
+          <param name="watchdog_timeout">0.5</param>
         </joint>
       </xacro:if>
@@ -23,5 +23,5 @@
           <param name="axis">1</param>
           <param name="enable_watchdog">1</param>
-          <param name="watchdog_timeout">0.1</param>
+          <param name="watchdog_timeout">0.5</param>
         </joint>
       </xacro:if>

File: odrive_demo_description/urdf/odrive.urdf.xacro (robot description, xacro)
@@ -10,5 +10,5 @@
       <parent link="world"/>
       <child link="link0"/>
-      <axis xyz="0 0 1"/>
+      <axis xyz="1.0 0.0 0.0"/>
     </joint>
   </xacro:if>
@@ -18,5 +18,5 @@
       <parent link="world"/>
       <child link="link1"/>
-      <axis xyz="0 0 1"/>
+      <axis xyz="1.0 0.0 0.0"/>
     </joint>
   </xacro:if>
